File: hardware/usbtomidi.brd (EAGLE design)
At the start: 50 x 38 mm, 45 parts, among them Q1 IRLML6246, Q2 IRLML6246, Q3 IRLML6246, Q4 IRLML6246, U1 SPX5205 3v3, X1 MOLEX_2HORIZONTAL, X3 MOLEX_6HORIZONTAL, Y1 32768Hz CFPX-217 12.5pF

Commit message: latest
Parts:
- U$6: value TXB0108 -> ADG3304; device Simplex-ICs:TSSOP20 -> Simplex-ICs:TSSOP14
- moved U$5 258.5 mm to (76.0, 55.1), turned to 270 degrees
- moved U$4 258.3 mm to (76.1, 63.6), turned to 270 degrees
- moved U$3 198.9 mm to (27.7, 34.0)
- moved U$8 187.4 mm to (18.9, 33.7)
- moved U$9 173.8 mm to (37.3, 9.49)
- moved Q4 116.8 mm to (61.0, 41.9), turned to 270 degrees
- moved R4 115.6 mm to (65.9, 41.9)
- moved Q3 106.7 mm to (61.1, 38.2), turned to 270 degrees
- moved R3 106.5 mm to (65.9, 38.9)
- moved U$6 99.2 mm to (-7.75, 6.01)
- moved R1 98.2 mm to (65.9, 35.9)
- moved Q1 97.0 mm to (61.1, 34.0), turned to 270 degrees
- moved OK1 93.8 mm to (73.4, 38.7)
- moved R26 90.7 mm to (65.9, 32.1)
- moved Q2 88.9 mm to (61.0, 30.4), turned to 270 degrees
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Connections:
- removed net 1: U$9.1
- removed net 4: U$9.4
- removed net SH: U$9.SH@1, U$9.SH@2, U$9.SH@3
- new net 5V_PC: U$10.1, U$10.15, U$10.8, U$10.9, U$4.13, U$4.3, U$5.13, U$5.3
- new net J1X: U$10.3, U$4.12
- new net J1Y: U$10.6, U$4.4
- new net J2X: U$10.11, U$5.12
- new net J2Y: U$10.13, U$5.4
- new net N$10: U$4.9
- new net N$11: U$4.7
- new net N$16: U$5.8
- new net N$17: U$5.9
- new net N$18: U$5.7
- new net N$4: U$4.8
- net +5V: now also U$4.11, U$5.11
- net B1: now also U$10.2
- net B2: now also U$10.7
- net B3: now also U$10.10
- net B4: now also U$10.14
- net GND: now also OK1.11, OK1.13, OK1.15, U$10.12, U$10.4, U$10.5, U$10.SH@1, U$10.SH@2, U$4.1, U$5.1, U$6.7
Other:
- board size 50 x 38 mm -> 100 x 100 mm

Commit message: latest
Parts:
- added C11, C12, C13: 100nF, rcl:C0805
- added C7: 1uF, rcl:C0805
- added U$11: SJ_3P, Simplex-Jumpers:SJ_3P
- moved U$6 93.7 mm to (65.2, 64.8), turned to 270 degrees
- moved X1 38.6 mm to (63.2, 28.6), turned to 0 degrees
- moved Q2 3.77 mm to (62.0, 34.0)
- moved Q1 3.33 mm to (62.0, 37.2)
- moved R26 2.56 mm to (66.6, 34.6)
- moved Q3 2.40 mm to (62.0, 40.4)
- moved Q4 1.98 mm to (62.0, 43.6)
- moved R1 1.68 mm to (66.6, 37.4)
- moved R3 1.48 mm to (66.6, 40.2)
- moved R4 1.35 mm to (66.6, 43.0)
- moved U$4 1.24 mm to (76.0, 64.8)
- moved U$5 0.46 mm to (76.0, 54.6)
- moved OK1 0.11 mm to (73.4, 38.8)
Connections:
- removed net 5V: X1.2
- removed net N$10: U$4.9
- removed net N$11: U$4.7
- removed net N$16: U$5.8
- removed net N$17: U$5.9
- removed net N$18: U$5.7
- removed net N$4: U$4.8
- removed net P4.0: R8.2, U$1.29, X3.2
- removed net P4.1: R7.2, U$1.30, X3.1
- new net 5V_EXT: U$11.3, X1.2
- new net HIGH_CS1: U$4.7, U$6.13
- new net HIGH_CS2: U$5.7, U$6.12
- new net HIGH_MOSI: U$4.8, U$5.8, U$6.11
- new net HIGH_SCLK: U$4.9, U$5.9, U$6.10
- new net RX: R8.2, U$1.34, X3.2
- new net SCLK: U$1.32
- new net TX: R7.2, U$1.33, X3.1
- net +3V3: now also U$6.1
- net +5V: now also C11.2, C12.2, C13.2, C7.2, U$11.2, U$6.14
- net 5V_PC: now also U$11.1
- net GND: now also C11.1, C12.1, C13.1, C7.1, U$9.SH@1, U$9.SH@2, U$9.SH@3
- net MISO: now also U$1.31; no longer U$1.34
- net MOSI: now also U$1.30; no longer U$1.33
Routing:
- net B3: track 0.00 -> 36.1 mm, vias 0 -> 2
- net +5V: track 0.00 -> 30.1 mm
- net HIGH_SCLK: track 0.00 -> 22.8 mm
- net HIGH_MOSI: track 0.00 -> 22.6 mm, vias 0 -> 2
- net B4: track 0.00 -> 18.9 mm
- net 5V_PC: track 0.00 -> 16.4 mm, vias 0 -> 1
- net HIGH_CS1: track 0.00 -> 14.4 mm
- net HIGH_CS2: track 0.00 -> 12.4 mm, vias 0 -> 2
- net B2: track 0.00 -> 5.95 mm
- net N$15: track 0.00 -> 2.93 mm
- net N$13: track 0.00 -> 2.82 mm
- net N$7: track 0.00 -> 2.72 mm
- net N$22: track 0.00 -> 2.70 mm
- net N$14: track 0.00 -> 2.70 mm
- net N$9: track 0.00 -> 2.61 mm
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