File: hardware/usbtomidi.sch (EAGLE design)
At the start: 45 parts, among them Q1 IRLML6246, Q2 IRLML6246, Q3 IRLML6246, Q4 IRLML6246, U1 SPX5205 3v3, X1 MOLEX_2HORIZONTAL, X3 MOLEX_6HORIZONTAL, Y1 32768Hz CFPX-217 12.5pF

Commit message: latest
Parts:
- U$6: value TXB0108 -> ADG3304; device Simplex-ICs:TXB0108 -> Simplex-ICs:ADG3304
Connections:
- new net 5V_PC: U$10.1, U$10.15, U$10.8, U$10.9, U$4.HA, U$4.HB, U$5.HA, U$5.HB
- new net J1X: U$10.3, U$4.WA
- new net J1Y: U$10.6, U$4.WB
- new net J2X: U$10.11, U$5.WA
- new net J2Y: U$10.13, U$5.WB
- new net N$10: U$4.SCLK
- new net N$11: U$4.!CS
- new net N$16: U$5.DIN
- new net N$17: U$5.SCLK
- new net N$18: U$5.!CS
- new net N$4: U$4.DIN
- net +5V: now also U$4.VDD, U$5.VDD
- net B1: now also U$10.2
- net B2: now also U$10.7
- net B3: now also U$10.10
- net B4: now also U$10.14
- net GND: now also OK1A.EMIT, OK1B.EMIT, OK1C.EMIT, U$10.12, U$10.4, U$10.5, U$10.SHIELD, U$4.GND, U$5.GND, U$6.GND
Other:
- moved on the sheet: C10, C17, C2, C23, C24, C5, C8, C9, OK1A, OK1B, OK1C, OK1D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

Commit message: latest
Parts:
- added C11, C12, C13: 100nF, rcl:C-EUC0805
- added C7: 1uF, rcl:C-EUC0805
- added U$11: SJ_3P, Simplex-Jumpers:SJ_3P
Connections:
- removed net 5V: X1.1
- removed net N$10: U$4.SCLK
- removed net N$11: U$4.!CS
- removed net N$16: U$5.DIN
- removed net N$17: U$5.SCLK
- removed net N$18: U$5.!CS
- removed net N$4: U$4.DIN
- removed net P4.0: R8.2, U$1.29, X3.5
- removed net P4.1: R7.2, U$1.30, X3.6
- new net 5V_EXT: U$11.3, X1.1
- new net HIGH_CS1: U$4.!CS, U$6.Y1
- new net HIGH_CS2: U$5.!CS, U$6.Y2
- new net HIGH_MOSI: U$4.DIN, U$5.DIN, U$6.Y3
- new net HIGH_SCLK: U$4.SCLK, U$5.SCLK, U$6.Y4
- new net RX: R8.2, U$1.34, X3.5
- new net SCLK: U$1.32
- new net TX: R7.2, U$1.33, X3.6
- net +3V3: now also U$6.VCCA
- net +5V: now also C11.2, C12.2, C13.2, C7.2, U$11.2, U$6.VCCY
- net 5V_PC: now also U$11.1
- net GND: now also C11.1, C12.1, C13.1, C7.1, U$9.SH
- net MISO: now also U$1.31; no longer U$1.34
- net MOSI: now also U$1.30; no longer U$1.33
Other:
- moved on the sheet: OK1A, OK1B, OK1C, OK1D, Q1, Q2, Q3, Q4, R1, R26, R3, R4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
