File: hardware/lemidi.brd (EAGLE design)
At the start: 100 x 100 mm, 66 parts, among them Q1 IRLML6246, Q2 IRLML6246, Q3 IRLML6246, Q4 IRLML6246, U1 SPX5205 3v3, X1 MOLEX_2HORIZONTAL, X3 MOLEX_6HORIZONTAL, Y1 32768Hz CFPX-217 12.5pF, Y2 12MHz 0.25%, Y3 8MHz

Commit message: happy new year
Parts:
- removed C23, C24: 22pF, rcl:C0805
- removed Y1: 32768Hz CFPX-217 12.5pF, Simplex-FreqCtrl:CRYSTAL-SMD-3.2X1.5
- moved U$7 112.4 mm to (71.8, 4.35), flipped to the bottom, turned to 90 degrees
- moved TP1 96.5 mm to (1.20, 7.40)
- moved TP3 87.6 mm to (6.40, 23.8)
- moved R10 81.3 mm to (3.40, 23.4), turned to 180 degrees
- moved TP2 75.8 mm to (6.60, 28.0)
- moved LED3 74.3 mm to (3.40, 21.2), turned to 90 degrees
- moved R9 69.6 mm to (3.40, 27.8), turned to 180 degrees
- moved LED2 62.6 mm to (3.40, 25.6), turned to 90 degrees
- moved C19 59.5 mm to (14.2, 33.8), turned to 270 degrees
- moved TP101 54.5 mm to (1.20, 7.40)
- moved C20 49.5 mm to (10.2, 18.4), turned to 270 degrees
- moved R4 41.5 mm to (43.4, 8.60), turned to 270 degrees
- moved Y3 41.0 mm to (28.0, 38.2)
- moved R3 40.9 mm to (40.6, 8.60), turned to 270 degrees
- moved R26 40.8 mm to (35.2, 8.60), turned to 270 degrees
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Connections:
- net N$1 renamed 12MHZ_XO
- net N$3 renamed 12MHX_XI
- removed net N$25: C24.1, U$1.9, Y1.P$1
- removed net N$26: C23.1, U$1.8, Y1.P$2
- removed net VIN: C3.1, C6.1, U1.1, U1.3
- new net N$1: LED1.A, R6.2
- new net N$20: U$1.20, U$2.2
- new net N$21: U$1.21, U$2.1
- new net N$3: U$1.18, U$2.4
- net +5V: now also C3.1, C6.1, U1.1, U1.3
- net B1_EN: now also U$2.8
- net B2_EN: now also U$2.7
- net B3_EN: now also U$2.6
- net B4_EN: now also U$2.5
- net GND: now also LED1.C, LED2.C, LED3.C; no longer C23.2, C24.2, R10.2, R6.2, R9.2
- net N$11: now also LED3.A, R10.2; no longer LED3.C, R10.1
- net N$4: now also LED2.A, R9.2; no longer LED2.C, R9.1
- net N$8: now also U$1.19, U$2.3; no longer LED1.C, R6.1
- net STATUS: now also R6.1; no longer LED1.A
- net USB_GPX: now also U$1.15
- net USB_INT: now also U$1.14
- net USB_ST1: now also R9.1; no longer LED2.A
- net USB_ST2: now also R10.1; no longer LED3.A
Routing:
- net +5V: track 30.1 -> 102.3 mm, vias 0 -> 2
- net VBUS: track 0.00 -> 25.7 mm, vias 0 -> 2
- net 12MHZ_XO: track 0.00 -> 22.2 mm
- net +3V3: track 0.00 -> 21.8 mm
- net N$21: track 0.00 -> 15.7 mm
- net N$20: track 0.00 -> 15.3 mm
- net N$8: track 0.00 -> 14.9 mm
- net N$3: track 0.00 -> 14.5 mm
- net 12MHX_XI: track 0.00 -> 13.5 mm
- net N$9: track 2.61 -> 14.4 mm
- net N$7: track 2.72 -> 12.6 mm
- net 5V_EXT: track 0.00 -> 9.18 mm
- net N$13: track 2.82 -> 11.5 mm
- net 5V_PC: track 16.4 -> 23.0 mm
- net B1_EN: track 0.00 -> 6.17 mm
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Other:
- board size 100 x 100 mm -> 76 x 42 mm
- board text added: "github.com/rodan/lemidi"
- board text removed: "+3V3"
- board text removed: "github.com/rodan/retrojoy"
- board text removed: "status"
- board text removed: "tp1"
- board text removed: "tp2"
- board text removed: "tp3"
- board text removed: "tp4"
- board text removed: "tp5"
- board text removed: "tp6"

Commit message: latest
Parts:
- LED3: value green -> red
- U$10: value ADAM_TECH-DSUB_DA-15 -> DA-15
- X1: value MOLEX_2HORIZONTAL -> optional 5V input
- X3: value MOLEX_6HORIZONTAL -> debug
- moved U$6 4.20 mm to (38.2, 35.0), turned to 0 degrees
- moved U$8 3.44 mm to (5.20, 14.6)
- moved C13 3.21 mm to (43.8, 37.2), turned to 0 degrees
- moved TP2 3.01 mm to (6.40, 25.0)
- moved R6 2.80 mm to (3.40, 29.4)
- moved LED1 2.80 mm to (3.40, 27.2)
- moved LED2 2.80 mm to (3.40, 22.8)
- moved LED3 2.80 mm to (3.40, 18.4)
- moved R9 2.80 mm to (3.40, 25.0)
- moved TP3 2.80 mm to (6.40, 21.0)
- moved TP6 2.80 mm to (6.93, 28.9)
- moved R10 2.80 mm to (3.40, 20.6)
- moved C2 2.61 mm to (38.2, 37.2)
- moved X3 2.60 mm to (4.60, 38.4)
- moved Y3 1.20 mm to (28.0, 37.0)
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Connections:
- removed net CSJ1: U$6.2
- removed net CSJ2: U$6.3
- removed net USB_CS: U$3.14
- new net CS_J1: U$1.36, U$6.2
- new net CS_J2: U$1.35, U$6.3
- new net CS_USB: U$1.29, U$3.14
- net HIGH_MOSI: now also U$6.10; no longer U$6.11
- net HIGH_SCLK: now also U$6.11; no longer U$6.10
- net MOSI: now also U$6.5; no longer U$6.4
- net SCLK: now also U$6.4; no longer U$6.5
- net USB_RES: now also U$1.2
Routing:
- net MOSI: track 0.00 -> 36.5 mm, vias 0 -> 2
- net SCLK: track 0.00 -> 34.7 mm, vias 0 -> 2
- net MISO: track 0.00 -> 24.1 mm, vias 0 -> 2
- net HIGH_MOSI: track 22.6 -> 13.8 mm
- net HIGH_CS1: track 14.4 -> 6.18 mm
- net HIGH_SCLK: track 22.8 -> 15.1 mm
- net +5V: track 102.3 -> 97.2 mm
- net N$11: track 0.00 -> 3.07 mm
- net N$4: track 0.00 -> 3.07 mm
- net N$1: track 0.00 -> 3.07 mm
- net STATUS: track 0.00 -> 2.67 mm
- net USB_ST2: track 0.00 -> 2.11 mm
- net USB_ST1: track 0.00 -> 1.95 mm
- net VBUS: track 25.7 -> 27.7 mm
- net GND: track 2.12 -> 3.72 mm, vias 9 -> 12
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Other:
- board size 76 x 42 mm -> 76 x 40 mm

Commit message: latest
Parts:
- added C21: 100nF, rcl:C0805
- added TP4, TP5: (no value), testpad:TP12R
- TP2, TP3, TP6: value TPTP12R -> (none)
- moved TP6 31.4 mm to (38.0, 24.6), flipped to the bottom, turned to 0 degrees
- moved TP2 29.6 mm to (35.2, 32.0), flipped to the bottom
- moved R7 11.1 mm to (16.0, 35.4), turned to 0 degrees
- moved R34 10.8 mm to (8.80, 35.4)
- moved C14 10.6 mm to (8.80, 33.2), turned to 180 degrees
- moved R8 6.93 mm to (16.0, 37.6), turned to 0 degrees
- moved TP3 6.37 mm to (10.8, 25.6), flipped to the bottom
- moved R35 4.40 mm to (8.80, 37.6), turned to 0 degrees
- moved C19 1.90 mm to (16.0, 33.2), turned to 180 degrees
Connections:
- removed net STATUS: R6.1, TP6.TP
- new net USB_ST3: R6.1, U$3.6
- net +3V3: now also C21.2
- net CS_USB: now also TP5.TP
- net GND: now also C21.1, TP6.TP
- net MISO: now also TP3.TP
- net MOSI: now also TP4.TP
- net SCLK: now also TP2.TP
- net USB_GPX: now also U$1.14; no longer U$1.15
- net USB_INT: now also U$1.15; no longer U$1.14
- net USB_ST1: no longer TP2.TP
- net USB_ST2: no longer TP3.TP
Routing:
- net +3V3: track 21.8 -> 101.8 mm, vias 0 -> 6
- net TX: track 0.00 -> 36.2 mm, vias 0 -> 2
- net RX: track 0.00 -> 33.0 mm, vias 0 -> 2
- net TEST: track 0.00 -> 29.7 mm, vias 0 -> 2
- net CS_USB: track 0.00 -> 29.5 mm, vias 0 -> 2
- net RST: track 0.00 -> 26.2 mm, vias 0 -> 2
- net VBUS_FLAG: track 0.00 -> 25.2 mm, vias 0 -> 2
- net USB_INT: track 0.00 -> 22.5 mm, vias 0 -> 2
- net VBUS_EN: track 0.00 -> 20.4 mm, vias 0 -> 2
- net USB_GPX: track 0.00 -> 17.1 mm, vias 0 -> 2
- net USB_RES: track 0.00 -> 16.1 mm, vias 0 -> 2
- net USB_ST2: track 2.11 -> 16.1 mm
- net GND: track 3.72 -> 17.4 mm, vias 12 -> 17
- net XT2IN: track 0.00 -> 12.3 mm
- net XT2OUT: track 0.00 -> 11.7 mm
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
Commit message: latest
Parts:
- moved C12 6.53 mm to (50.6, 18.6), turned to 180 degrees
- moved C7 0.80 mm to (50.6, 16.4)
- moved OK1 0.80 mm to (50.6, 10.0)
- moved C11 0.20 mm to (55.0, 34.0)
Routing:
- net 5V_PC: track 23.6 -> 81.3 mm, vias 1 -> 7
- net +5V: track 94.6 -> 137.1 mm, vias 2 -> 5
- net J1Y: track 0.00 -> 42.1 mm, vias 0 -> 2
- net J2Y: track 0.00 -> 18.4 mm, vias 0 -> 2
- net B1: track 0.00 -> 15.3 mm, vias 0 -> 1
- net J1X: track 0.00 -> 13.4 mm
- net J2X: track 0.00 -> 13.0 mm
- net HIGH_MOSI: track 13.8 -> 20.3 mm
- net HIGH_SCLK: track 15.1 -> 19.8 mm
- net HIGH_CS1: track 3.55 -> 6.32 mm
- net HIGH_CS2: track 7.50 -> 10.1 mm
- net N$15: track 8.85 -> 8.05 mm
- net GND: vias 17 -> 23

Commit message: ERC pass
Parts:
- C14: value 10nF -> 2.2nF
Connections:
- removed net N$10: U$3.3
- net GND: now also U$3.3
Changed lines of the file:
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@@
 <element name="C13" library="rcl" package="C0805" value="100nF" x="43.8" y="37.2"/>
 <element name="U$11" library="Simplex-Jumpers" package="SJ_3P" value="SJ_3P" x="44.8" y="2.2" rot="R180"/>
-<element name="C14" library="rcl" package="C0805" value="10nF" x="8.8" y="33.2" rot="R180"/>
+<element name="C14" library="rcl" package="C0805" value="2.2nF" x="8.8" y="33.2" rot="R180"/>
 <element name="Y2" library="Simplex-FreqCtrl" package="CRYSTAL-SMD-11.4X4.35" value="12MHz 0.25%" x="28" y="18.4"/>
 <element name="Y3" library="Simplex-FreqCtrl" package="CRYSTAL-SMD-11.4X4.35" value="8MHz" x="28" y="37" rot="R180"/>
@@
 <via x="55" y="10.6" extent="1-16" drill="0.4"/>
 <via x="55" y="13.2" extent="1-16" drill="0.4"/>
+<contactref element="U$3" pad="3"/>
+<wire x1="18.2" y1="29" x2="14.56" y2="29.53" width="0" layer="19" extent="1-1"/>
 </signal>
 <signal name="+3V3">
@@
 <wire x1="11.6" y1="26.6" x2="12" y2="27.2" width="0.3048" layer="1"/>
 </signal>
-<signal name="N$10">
-<contactref element="U$3" pad="3"/>
-</signal>
 <signal name="USB_INT">

Commit message: DRC pass
Routing:
- net GND: track 17.4 -> 21.1 mm, vias 23 -> 24
Changed lines of the file:
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@@
 </class>
 </classes>
-<designrules name="seeedstudio_rules_v1.1 *">
+<designrules name="seeed_2-layer_20140221">
 <description language="de">&lt;b&gt;EAGLE Design Rules&lt;/b&gt;
 &lt;p&gt;
@@
 </description>
 <param name="layerSetup" value="(1*16)"/>
-<param name="mtCopper" value="0.035mm 0.035mm 0.035mm 0.035mm 0.035mm 0.035mm 0.035mm 0.035mm 0.035mm 0.035mm 0.035mm 0.035mm 0.035mm 0.035mm 0.035mm 0.035mm"/>
-<param name="mtIsolate" value="1.5mm 0.15mm 0.2mm 0.15mm 0.2mm 0.15mm 0.2mm 0.15mm 0.2mm 0.15mm 0.2mm 0.15mm 0.2mm 0.15mm 0.2mm"/>
+<param name="mtCopper" value="0.035mm 0.0175mm 0.035mm 0.035mm 0.035mm 0.035mm 0.035mm 0.035mm 0.035mm 0.035mm 0.035mm 0.035mm 0.035mm 0.035mm 0.0175mm 0.035mm"/>
+<param name="mtIsolate" value="1.5mm 1.1mm 0.2mm 0.15mm 0.2mm 0.15mm 0.2mm 0.15mm 0.2mm 0.15mm 0.2mm 0.15mm 0.2mm 0.15mm 0.2mm"/>
 <param name="mdWireWire" value="6mil"/>
 <param name="mdWirePad" value="6mil"/>
@@
 <param name="rvMicroViaOuter" value="0.25"/>
 <param name="rvMicroViaInner" value="0.25"/>
-<param name="rlMinPadTop" value="0.154mm"/>
+<param name="rlMinPadTop" value="6mil"/>
 <param name="rlMaxPadTop" value="20mil"/>
-<param name="rlMinPadInner" value="0.154mm"/>
+<param name="rlMinPadInner" value="10mil"/>
 <param name="rlMaxPadInner" value="20mil"/>
-<param name="rlMinPadBottom" value="0.154mm"/>
+<param name="rlMinPadBottom" value="6mil"/>
 <param name="rlMaxPadBottom" value="20mil"/>
 <param name="rlMinViaOuter" value="6mil"/>
@@
 <contactref element="U$1" pad="10"/>
 <via x="18.2" y="29" extent="1-16" drill="0.4"/>
-<wire x1="13.06" y1="23.21" x2="13.06" y2="21.86" width="0.3048" layer="1"/>
-<wire x1="13.06" y1="21.86" x2="12.6" y2="21.4" width="0.3048" layer="1"/>
+<wire x1="13.06" y1="23.21" x2="13.06" y2="21.66" width="0.3048" layer="1"/>
 <contactref element="LED2" pad="C"/>
 <contactref element="LED3" pad="C"/>
 <via x="26.2" y="8.6" extent="1-16" drill="0.4"/>
-<via x="11.8" y="21.4" extent="1-16" drill="0.4"/>
+<via x="10.2" y="21.2" extent="1-16" drill="0.4"/>
 <via x="4" y="15.6" extent="1-16" drill="0.4"/>
 <via x="24.6" y="21.6" extent="1-16" drill="0.4"/>
@@
 <wire x1="33.1" y1="27.05" x2="31.85" y2="27.05" width="0.3048" layer="1"/>
 <wire x1="31.85" y1="27.05" x2="31.6" y2="26" width="0.3048" layer="1"/>
-<wire x1="11.8" y1="21.4" x2="12.6" y2="21.4" width="0.3048" layer="1"/>
 <contactref element="C21" pad="1"/>
 <via x="26" y="26" extent="1-16" drill="0.4"/>
@@
 <via x="55" y="13.2" extent="1-16" drill="0.4"/>
 <contactref element="U$3" pad="3"/>
-<wire x1="18.2" y1="29" x2="14.56" y2="29.53" width="0" layer="19" extent="1-1"/>
+<via x="14" y="31.2" extent="1-16" drill="0.4"/>
+<wire x1="14.56" y1="29.53" x2="14.56" y2="30.64" width="0.3048" layer="1"/>
+<wire x1="14.56" y1="30.64" x2="14" y2="31.2" width="0.3048" layer="1"/>
+<wire x1="13.06" y1="21.66" x2="12.6" y2="21.2" width="0.3048" layer="1"/>
+<wire x1="12.6" y1="21.2" x2="10.2" y2="21.2" width="0.3048" layer="1"/>
 </signal>
 <signal name="+3V3">
@@
 <wire x1="15.06" y1="23.21" x2="15.06" y2="25.34" width="0.3048" layer="1"/>
 <wire x1="15.06" y1="25.34" x2="14.6" y2="25.8" width="0.3048" layer="1"/>
-<wire x1="14.6" y1="25.8" x2="14.6" y2="27.8" width="0.3048" layer="1"/>
-<wire x1="14.6" y1="27.8" x2="15.06" y2="28.26" width="0.3048" layer="1"/>
-<wire x1="15.06" y1="28.26" x2="15.06" y2="29.53" width="0.3048" layer="1"/>
+<wire x1="14.6" y1="25.8" x2="14.6" y2="28" width="0.3048" layer="1"/>
+<wire x1="14.6" y1="28" x2="15.06" y2="28.46" width="0.3048" layer="1"/>
+<wire x1="15.06" y1="28.46" x2="15.06" y2="29.53" width="0.3048" layer="1"/>
 <wire x1="19.2" y1="20.2" x2="18.8" y2="20.6" width="0.4064" layer="1"/>
 <wire x1="15.06" y1="29.53" x2="15.06" y2="33.19" width="0.3048" layer="1"/>
@@
 <wire x1="25.8" y1="23.4" x2="26" y2="23.2" width="0.3048" layer="16"/>
 <via x="26" y="23.2" extent="1-16" drill="0.4"/>
-<wire x1="26.55" y1="24.5" x2="26.55" y2="23.75" width="0.3048" layer="1"/>
-<wire x1="26.55" y1="23.75" x2="26" y2="23.2" width="0.3048" layer="1"/>
+<wire x1="26.55" y1="24.5" x2="26.55" y2="23.2" width="0.3048" layer="1"/>
 <wire x1="12.06" y1="23.21" x2="11.61" y2="23.21" width="0.3048" layer="1"/>
 <wire x1="11.61" y1="23.21" x2="11.4" y2="23" width="0.3048" layer="1"/>
+<wire x1="26.55" y1="23.2" x2="26" y2="23.2" width="0.3048" layer="1"/>
 </signal>
 <signal name="N$16">
@@
 <contactref element="R2" pad="1"/>
 <contactref element="U$3" pad="20"/>
-<wire x1="13.56" y1="21.56" x2="13.56" y2="23.21" width="0.3048" layer="1"/>
-<wire x1="13.56" y1="21.56" x2="13" y2="21" width="0.3048" layer="1"/>
-<wire x1="13" y1="21" x2="13" y2="19.4525" width="0.3048" layer="1"/>
+<wire x1="13.56" y1="21.36" x2="13.56" y2="23.21" width="0.3048" layer="1"/>
+<wire x1="13.56" y1="21.36" x2="13" y2="20.8" width="0.3048" layer="1"/>
+<wire x1="13" y1="20.8" x2="13" y2="19.4525" width="0.3048" layer="1"/>
 </signal>
 <signal name="D+">
@@
 <contactref element="U$8" pad="4"/>
 <wire x1="15.56" y1="29.53" x2="15.56" y2="27.6" width="0.3048" layer="1"/>
-<wire x1="15.56" y1="27.6" x2="15.4" y2="27.4" width="0.3048" layer="1"/>
-<via x="15.4" y="27.4" extent="1-16" drill="0.4"/>
-<wire x1="15.4" y1="27.4" x2="13" y2="27.4" width="0.3048" layer="16"/>
+<wire x1="15.56" y1="27.6" x2="15.4" y2="27.6" width="0.3048" layer="1"/>
+<via x="15.4" y="27.6" extent="1-16" drill="0.4"/>
 <wire x1="13" y1="27.4" x2="12.4" y2="28" width="0.3048" layer="16"/>
 <wire x1="12.4" y1="28" x2="11.6" y2="28" width="0.3048" layer="16"/>
@@
 <wire x1="8.4" y1="26" x2="8.4" y2="20" width="0.3048" layer="16"/>
 <wire x1="8.4" y1="20" x2="8.6" y2="19.8" width="0.3048" layer="16"/>
+<wire x1="13" y1="27.4" x2="15.2" y2="27.4" width="0.3048" layer="16"/>
+<wire x1="15.2" y1="27.4" x2="15.4" y2="27.6" width="0.3048" layer="16"/>
 </signal>
 <signal name="N$18">

Commit message: 1st cleanup
Parts:
- added TP7: (no value), testpad:TP12R
- moved TP6 1.81 mm to (36.2, 24.4)
- moved TP2 1.00 mm to (36.2, 32.0)
- moved TP1 0.20 mm to (1.40, 7.40)
- moved TP101 0.20 mm to (1.40, 7.40)
Connections:
- net CS_J1: now also TP7.TP
Routing:
- net CS_J1: track 6.61 -> 8.12 mm, vias 0 -> 1
- net 5V_PC: track 81.3 -> 82.8 mm
- net GND: vias 24 -> 35
Other:
- board text added: "J1"
- board text added: "Petre Rodan 201901 rev1"
- board text added: "opt 5V"
- board text removed: "5V"
- board text removed: "Petre Rodan 201812 rev1"
Changed lines of the file:
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@@
 <grid distance="0.2" unitdist="mm" unit="mm" style="dots" multiple="1" display="no" altdistance="0.635" altunitdist="mm" altunit="mm"/>
 <layers>
-<layer number="1" name="Top" color="4" fill="1" visible="yes" active="yes"/>
+<layer number="1" name="Top" color="4" fill="1" visible="no" active="yes"/>
 <layer number="2" name="Route2" color="1" fill="3" visible="no" active="no"/>
 <layer number="3" name="Route3" color="4" fill="3" visible="no" active="no"/>
@@
 <hole x="3.1" y="3.1" drill="3.2"/>
 <rectangle x1="19.7" y1="6.5" x2="21.2" y2="8" layer="30"/>
-<text x="35.27" y="0.77" size="0.8128" layer="108" font="vector" ratio="15">5V</text>
+<text x="34.73" y="0.97" size="0.8128" layer="109" font="vector" ratio="15" rot="MR0">opt 5V</text>
 <text x="1.8" y="9.4" size="1.016" layer="1" font="vector" ratio="15" rot="R90">1</text>
 <text x="1.8" y="11.2" size="1.016" layer="16" font="vector" ratio="15" rot="R90">2</text>
 <text x="70.3" y="8.13" size="0.8128" layer="109" font="vector" ratio="15" rot="MR90">github.com/rodan/lemidi</text>
-<text x="71.73" y="8.15" size="0.8128" layer="109" font="vector" ratio="15" rot="MR90">Petre Rodan 201812 rev1</text>
-<text x="2.23" y="36.83" size="0.8128" layer="108" font="vector" ratio="15" rot="MR270">debug</text>
+<text x="71.93" y="8.15" size="0.8128" layer="109" font="vector" ratio="15" rot="MR90">Petre Rodan 201901 rev1</text>
+<text x="2.23" y="36.83" size="0.8128" layer="109" font="vector" ratio="15" rot="MR270">debug</text>
 <wire x1="1.35" y1="9.35" x2="1.35" y2="12.15" width="1.6764" layer="41"/>
 <rectangle x1="17.8" y1="5.1" x2="21.8" y2="9.4" layer="30"/>
+<text x="46" y="0.6" size="0.8128" layer="108" ratio="15">J1</text>
 </plain>
 <attributes>
@@
 <attribute name="TP_SIGNAL_NAME" value="" x="23.84" y="11.36" size="1.778" layer="27" rot="R270" display="off"/>
 </element>
-<element name="TP1" library="testpad" package="TP12R" value="TPTP12R" x="1.2" y="7.4" rot="R180">
-<attribute name="TP_SIGNAL_NAME" value="" x="1.2" y="7.4" size="1.778" layer="27" rot="R180" display="off"/>
+<element name="TP1" library="testpad" package="TP12R" value="TPTP12R" x="1.4" y="7.4" rot="R180">
+<attribute name="TP_SIGNAL_NAME" value="" x="1.4" y="7.4" size="1.778" layer="27" rot="R180" display="off"/>
 </element>
-<element name="TP101" library="testpad" package="TP12R" value="TPTP12R" x="1.2" y="7.4" rot="MR180">
-<attribute name="TP_SIGNAL_NAME" value="" x="1.2" y="7.4" size="1.778" layer="28" rot="MR180" display="off"/>
+<element name="TP101" library="testpad" package="TP12R" value="TPTP12R" x="1.4" y="7.4" rot="MR180">
+<attribute name="TP_SIGNAL_NAME" value="" x="1.4" y="7.4" size="1.778" layer="28" rot="MR180" display="off"/>
 </element>
 <element name="C3" library="rcl" package="C0805" value="10uF" x="26.55" y="3.33"/>
@@
 <element name="LED3" library="led" package="CHIPLED_0805" value="red" x="3.4" y="18.4" rot="R90"/>
 <element name="C21" library="rcl" package="C0805" value="100nF" x="41" y="29" rot="R180"/>
-<element name="TP2" library="testpad" package="TP12R" value="" x="35.2" y="32" rot="MR0">
-<attribute name="TP_SIGNAL_NAME" value="" x="35.2" y="32" size="1.778" layer="28" rot="MR0" display="off"/>
+<element name="TP2" library="testpad" package="TP12R" value="" x="36.2" y="32" rot="MR0">
+<attribute name="TP_SIGNAL_NAME" value="" x="36.2" y="32" size="1.778" layer="28" rot="MR0" display="off"/>
 </element>
 <element name="TP3" library="testpad" package="TP12R" value="" x="10.8" y="25.6" rot="MR0">
@@
 <attribute name="TP_SIGNAL_NAME" value="" x="29.6" y="26.8" size="1.778" layer="28" rot="MR0" display="off"/>
 </element>
-<element name="TP6" library="testpad" package="TP12R" value="" x="38" y="24.6" rot="MR0">
-<attribute name="TP_SIGNAL_NAME" value="" x="38" y="24.6" size="1.778" layer="28" rot="MR0" display="off"/>
+<element name="TP6" library="testpad" package="TP12R" value="" x="36.2" y="24.4" rot="MR0">
+<attribute name="TP_SIGNAL_NAME" value="" x="36.2" y="24.4" size="1.778" layer="28" rot="MR0" display="off"/>
+</element>
+<element name="TP7" library="testpad" package="TP12R" value="" x="36.2" y="35.8" rot="MR0">
+<attribute name="TP_SIGNAL_NAME" value="" x="36.2" y="35.8" size="1.778" layer="28" rot="MR0" display="off"/>
 </element>
 </elements>
@@
 <wire x1="13.06" y1="21.66" x2="12.6" y2="21.2" width="0.3048" layer="1"/>
 <wire x1="12.6" y1="21.2" x2="10.2" y2="21.2" width="0.3048" layer="1"/>
+<via x="39.6" y="26.6" extent="1-16" drill="0.4"/>
+<via x="43.6" y="27.8" extent="1-16" drill="0.4"/>
+<via x="42.2" y="11.6" extent="1-16" drill="0.4"/>
+<via x="19.8" y="39" extent="1-16" drill="0.4"/>
+<via x="35.6" y="39" extent="1-16" drill="0.4"/>
+<via x="41" y="37.2" extent="1-16" drill="0.4"/>
+<via x="60.8" y="31.8" extent="1-16" drill="0.4"/>
+<via x="53.2" y="17.6" extent="1-16" drill="0.4"/>
+<via x="1.4" y="5.8" extent="1-16" drill="0.4"/>
+<via x="1" y="28.2" extent="1-16" drill="0.4"/>
+<via x="1" y="19.4" extent="1-16" drill="0.4"/>
 </signal>
 <signal name="+3V3">
@@
 <wire x1="63.495" y1="27" x2="65.2" y2="27" width="0.4064" layer="1"/>
 <via x="65.2" y="27" extent="1-16" drill="0.4"/>
-<via x="67.6" y="27" extent="1-16" drill="0.4"/>
-<wire x1="67.6" y1="27" x2="67.6" y2="12.4" width="0.4064" layer="1"/>
+<via x="67.2" y="28.2" extent="1-16" drill="0.4"/>
 <wire x1="67.6" y1="12.4" x2="66.8" y2="11.6" width="0.4064" layer="1"/>
-<wire x1="65.2" y1="27" x2="67.6" y2="27" width="0.4064" layer="16"/>
 <wire x1="60.825" y1="29.67" x2="62.21" y2="28.285" width="0.6096" layer="1"/>
 <via x="66.8" y="11.6" extent="1-16" drill="0.4"/>
 <wire x1="66.8" y1="11.6" x2="66.735" y2="11.665" width="0.4064" layer="16"/>
 <wire x1="66.735" y1="11.665" x2="62.21" y2="11.665" width="0.4064" layer="16"/>
+<wire x1="67.6" y1="12.4" x2="67.6" y2="27.6" width="0.4064" layer="1"/>
+<wire x1="65.2" y1="27" x2="66.4" y2="28.2" width="0.4064" layer="16"/>
+<wire x1="66.4" y1="28.2" x2="67.2" y2="28.2" width="0.4064" layer="16"/>
+<wire x1="67.6" y1="27.6" x2="67.2" y2="28" width="0.4064" layer="1"/>
+<wire x1="67.2" y1="28" x2="67.2" y2="28.2" width="0.4064" layer="1"/>
 </signal>
 <signal name="J1X">
@@
 <wire x1="12.2" y1="26.2" x2="17.4" y2="26.2" width="0.3048" layer="16"/>
 <contactref element="TP2" pad="TP"/>
-<wire x1="35.2" y1="32" x2="35.2" y2="31" width="0.3048" layer="16"/>
+<wire x1="36.2" y1="32" x2="35.2" y2="31" width="0.3048" layer="16"/>
 <wire x1="35.2" y1="31" x2="35.4" y2="30.8" width="0.3048" layer="16"/>
 </signal>
@@
 <wire x1="16.97" y1="24.62" x2="18.39" y2="23.2" width="0.3048" layer="1"/>
 <wire x1="18.39" y1="23.2" x2="19.2" y2="23.2" width="0.3048" layer="1"/>
-<wire x1="19.2" y1="23.2" x2="21.6" y2="20.8" width="0.3048" layer="1"/>
-<wire x1="21.6" y1="20.8" x2="27.8" y2="20.8" width="0.3048" layer="1"/>
-<wire x1="27.8" y1="20.8" x2="30.2" y2="18.4" width="0.3048" layer="1"/>
+<wire x1="19.2" y1="23.2" x2="22" y2="20.4" width="0.3048" layer="1"/>
 <wire x1="30.2" y1="18.4" x2="30.8" y2="18.4" width="0.3048" layer="1"/>
-<wire x1="30.8" y1="18.4" x2="32.75" y2="18.4" width="0.3048" layer="1"/>
+<wire x1="31.4" y1="18.4" x2="32.75" y2="18.4" width="0.3048" layer="1"/>
 <wire x1="30.75" y1="14.6" x2="30.8" y2="14.65" width="0.3048" layer="1"/>
 <wire x1="30.8" y1="14.65" x2="30.8" y2="18.4" width="0.3048" layer="1"/>
+<wire x1="22" y1="20.4" x2="28.2" y2="20.4" width="0.3048" layer="1"/>
+<wire x1="28.2" y1="20.4" x2="30.2" y2="18.4" width="0.3048" layer="1"/>
+<wire x1="30.8" y1="18.4" x2="31.4" y2="18.4" width="0.3048" layer="1"/>
 </signal>
 <signal name="12MHX_XI">
@@
 <wire x1="34.4" y1="32.4" x2="36.35" y2="34.35" width="0.3048" layer="1"/>
 <wire x1="36.35" y1="34.35" x2="38.2" y2="34.35" width="0.3048" layer="1"/>
+<contactref element="TP7" pad="TP"/>
+<wire x1="36.2" y1="35.8" x2="36.2" y2="34.8" width="0.3048" layer="16"/>
+<via x="36.2" y="34.8" extent="1-16" drill="0.4"/>
+<wire x1="36.35" y1="34.35" x2="36.35" y2="34.65" width="0.3048" layer="1"/>
+<wire x1="36.35" y1="34.65" x2="36.2" y2="34.8" width="0.3048" layer="1"/>
 </signal>
 <signal name="CS_J2">
