File: hardware/lemidi.brd (EAGLE design)
At the start: 76 x 40 mm, 67 parts, among them Q1 IRLML6246, Q2 IRLML6246, Q3 IRLML6246, Q4 IRLML6246, U1 SPX5205 3v3, X1 optional 5V input, X3 debug, Y2 12MHz 0.25%, Y3 8MHz

Commit message: 2nd cleanup
Parts:
- moved TP7 27.4 mm to (10.8, 25.6)
- moved TP3 25.5 mm to (36.2, 28.2)
- moved TP5 11.2 mm to (36.2, 35.8)
- moved TP2 7.60 mm to (36.2, 24.4)
- moved TP6 7.02 mm to (29.6, 26.8)
- moved TP4 3.80 mm to (36.2, 32.0)
Connections:
- removed net CS_J1: TP7.TP, U$1.36, U$6.2
- new net TP5: TP5.TP, U$1.36, U$6.2
- net CS_USB: now also TP6.TP; no longer TP5.TP
- net GND: now also TP2.TP; no longer TP6.TP
- net MISO: now also TP7.TP; no longer TP3.TP
- net MOSI: now also TP3.TP; no longer TP4.TP
- net SCLK: now also TP4.TP; no longer TP2.TP
Routing:
- net TP5: track 0.00 -> 8.12 mm, vias 0 -> 1
- net CS_J1: track 8.12 -> 0.00 mm, vias 1 -> 0
Other:
- board text added: "1-2 external 5V 2-3 (def) midi 5V"
- board text added: "J1 jumper"
- board text added: "ext 5V"
- board text added: "gnd"
- board text added: "rst"
- board text added: "rx"
- board text added: "test"
- board text added: "test points"
- board text added: "tp1"
- board text added: "tp1 - gnd tp2 - gnd tp3 - mosi tp4 - clk tp5 - cs J1 tp6 - cs usb tp7 - miso"
- board text added: "tp2"
- board text added: "tp3"
- board text added: "tp4"
- board text added: "tp5"
- board text added: "tp6"
- board text added: "tp7"
- board text added: "tx[]"
- board text added: "vcc"
- board text removed: "opt 5V"
