File: hardware/lemidi.brd (EAGLE design)
At the start: 76 x 40 mm, 71 parts, among them Q1 IRLML6246, Q2 IRLML6246, Q3 IRLML6246, Q4 IRLML6246, Q5 si2305cd, U1 SPX5205 3v3, X3 debug, Y2 12MHz 0.25% CL 16pF, Y3 8MHz CL 18pF

Commit message: latest
Routing:
- net J1Y: track 19.8 -> 20.8 mm
- net GND: vias 51 -> 52
Changed lines of the file:
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@@
 <layer number="39" name="tKeepout" color="4" fill="11" visible="yes" active="yes"/>
 <layer number="40" name="bKeepout" color="1" fill="11" visible="yes" active="yes"/>
-<layer number="41" name="tRestrict" color="4" fill="10" visible="yes" active="yes"/>
-<layer number="42" name="bRestrict" color="1" fill="10" visible="yes" active="yes"/>
+<layer number="41" name="tRestrict" color="4" fill="10" visible="no" active="yes"/>
+<layer number="42" name="bRestrict" color="1" fill="10" visible="no" active="yes"/>
 <layer number="43" name="vRestrict" color="2" fill="10" visible="no" active="yes"/>
 <layer number="44" name="Drills" color="7" fill="1" visible="no" active="yes"/>
@@
 <layer number="106" name="bPlate" color="7" fill="1" visible="no" active="yes"/>
 <layer number="107" name="Crop" color="7" fill="1" visible="no" active="yes"/>
-<layer number="108" name="tmine" color="14" fill="1" visible="no" active="yes"/>
-<layer number="109" name="bmine" color="13" fill="1" visible="no" active="yes"/>
+<layer number="108" name="tmine" color="14" fill="1" visible="yes" active="yes"/>
+<layer number="109" name="bmine" color="13" fill="1" visible="yes" active="yes"/>
 <layer number="110" name="fp0" color="7" fill="1" visible="no" active="yes"/>
 <layer number="111" name="LPC17xx" color="7" fill="1" visible="no" active="yes"/>
@@
 <via x="27" y="14.4" extent="1-16" drill="0.4"/>
 <via x="18.4" y="32.6" extent="1-16" drill="0.4"/>
+<via x="18.8" y="24.2" extent="1-16" drill="0.4"/>
 </signal>
 <signal name="+3V3">
@@
 <wire x1="56.8" y1="28.2" x2="57.8" y2="27.2" width="0.4064" layer="1"/>
 <wire x1="57.8" y1="27.2" x2="57.8" y2="24.6" width="0.4064" layer="1"/>
-<wire x1="52.28" y1="36.68" x2="52.28" y2="37.08" width="0.4064" layer="1"/>
 <wire x1="52.28" y1="37.08" x2="52.8" y2="37.6" width="0.4064" layer="1"/>
-<wire x1="52.28" y1="36.68" x2="52.28" y2="35.73" width="0" layer="19" extent="1-1"/>
+<wire x1="52.28" y1="37.08" x2="52.28" y2="35.73" width="0.4064" layer="1"/>
 </signal>
 <signal name="J2X">
@@
 <wire x1="44.15" y1="29.6" x2="45" y2="29.6" width="0.3048" layer="1"/>
 <via x="45.2" y="27.4" extent="1-16" drill="0.4"/>
-<wire x1="45" y1="29.6" x2="46" y2="28.6" width="0.3048" layer="1"/>
 <wire x1="46" y1="28.6" x2="49.2" y2="28.6" width="0.3048" layer="1"/>
 <via x="44.2" y="20.8" extent="1-16" drill="0.4"/>
@@
 <wire x1="49.4" y1="18.6" x2="49.74" y2="18.94" width="0.3048" layer="1"/>
 <wire x1="49.74" y1="18.94" x2="49.74" y2="20.2" width="0.3048" layer="1"/>
+<wire x1="45" y1="29.6" x2="46" y2="28.6" width="0.3048" layer="1"/>
 </signal>
 <signal name="HIGH_SCLK">
@@
 <contactref element="U$11" pad="2"/>
 <contactref element="U$4" pad="2"/>
-<wire x1="44.15" y1="30.25" x2="45.75" y2="30.25" width="0.3048" layer="1"/>
-<wire x1="46.6" y1="29.4" x2="48.2" y2="29.4" width="0.3048" layer="1"/>
+<wire x1="46.4" y1="29.4" x2="48.2" y2="29.4" width="0.3048" layer="1"/>
 <wire x1="48.2" y1="29.4" x2="48.47" y2="29.67" width="0.3048" layer="1"/>
 <wire x1="48.47" y1="29.67" x2="48.47" y2="31" width="0.3048" layer="1"/>
-<via x="45.8" y="29.8" extent="1-16" drill="0.4"/>
-<wire x1="45.75" y1="30.25" x2="46" y2="30" width="0.3048" layer="1"/>
-<wire x1="46" y1="30" x2="46.6" y2="29.4" width="0.3048" layer="1"/>
-<wire x1="45.8" y1="29.8" x2="46" y2="30" width="0.3048" layer="1"/>
+<via x="46" y="29.8" extent="1-16" drill="0.4"/>
 <via x="45.2" y="20.8" extent="1-16" drill="0.4"/>
 <wire x1="45.2" y1="20.8" x2="45.2" y2="20" width="0.3048" layer="1"/>
@@
 <wire x1="45.2" y1="20.8" x2="46" y2="21.6" width="0.3048" layer="16"/>
 <wire x1="46" y1="21.6" x2="46" y2="29.6" width="0.3048" layer="16"/>
-<wire x1="46" y1="29.6" x2="45.8" y2="29.8" width="0.3048" layer="16"/>
+<wire x1="45.9" y1="29.7" x2="46" y2="29.8" width="0.3048" layer="16"/>
+<wire x1="44.15" y1="30.25" x2="45.55" y2="30.25" width="0.3048" layer="1"/>
+<wire x1="45.55" y1="30.25" x2="46" y2="29.8" width="0.3048" layer="1"/>
+<wire x1="46" y1="29.6" x2="45.9" y2="29.7" width="0.3048" layer="16"/>
+<wire x1="45.9" y1="29.7" x2="45.9" y2="29.9" width="0.3048" layer="16"/>
+<wire x1="46.4" y1="29.4" x2="46" y2="29.8" width="0.3048" layer="1"/>
 </signal>
 <signal name="HIGH_CS1">
@@
 <via x="46.2" y="20.8" extent="1-16" drill="0.4"/>
 <wire x1="46.6" y1="20.8" x2="47.2" y2="20.2" width="0.3048" layer="1"/>
-<wire x1="46.2" y1="30.8" x2="46.6" y2="30.4" width="0.3048" layer="16"/>
-<wire x1="46.6" y1="30.4" x2="46.6" y2="21.2" width="0.3048" layer="16"/>
 <wire x1="46.6" y1="21.2" x2="46.2" y2="20.8" width="0.3048" layer="16"/>
 <wire x1="46.2" y1="20.8" x2="46.6" y2="20.8" width="0.3048" layer="1"/>
+<wire x1="46.2" y1="30.8" x2="46.4" y2="30.6" width="0.3048" layer="16"/>
+<wire x1="46.4" y1="30.6" x2="46.6" y2="30.6" width="0.3048" layer="16"/>
+<wire x1="46.6" y1="30.6" x2="46.8" y2="30.4" width="0.3048" layer="16"/>
+<wire x1="46.8" y1="30.4" x2="46.8" y2="29.2" width="0.3048" layer="16"/>
+<wire x1="46.8" y1="29.2" x2="46.6" y2="29" width="0.3048" layer="16"/>
+<wire x1="46.6" y1="29" x2="46.6" y2="21.2" width="0.3048" layer="16"/>
 </signal>
 <signal name="5V_EXT">

Commit message: latest
Parts:
- moved U$7 5.95 mm to (71.0, 8.95)
- moved J1 3.00 mm to (41.9, 2.00), turned to 0 degrees
Connections:
- net N$10: now also J1.3; no longer J1.1
- net N$23: now also J1.1; no longer J1.3
Routing:
- net N$10: track 4.45 -> 5.25 mm
Changed lines of the file:
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@@
 <layer number="29" name="tStop" color="7" fill="3" visible="no" active="yes"/>
 <layer number="30" name="bStop" color="7" fill="6" visible="no" active="yes"/>
-<layer number="31" name="tCream" color="7" fill="4" visible="yes" active="yes"/>
-<layer number="32" name="bCream" color="7" fill="5" visible="yes" active="yes"/>
+<layer number="31" name="tCream" color="7" fill="4" visible="no" active="yes"/>
+<layer number="32" name="bCream" color="7" fill="5" visible="no" active="yes"/>
 <layer number="33" name="tFinish" color="6" fill="3" visible="no" active="yes"/>
 <layer number="34" name="bFinish" color="6" fill="6" visible="no" active="yes"/>
@@
 <layer number="37" name="tTest" color="7" fill="1" visible="no" active="yes"/>
 <layer number="38" name="bTest" color="7" fill="1" visible="no" active="yes"/>
-<layer number="39" name="tKeepout" color="4" fill="11" visible="yes" active="yes"/>
-<layer number="40" name="bKeepout" color="1" fill="11" visible="yes" active="yes"/>
+<layer number="39" name="tKeepout" color="4" fill="11" visible="no" active="yes"/>
+<layer number="40" name="bKeepout" color="1" fill="11" visible="no" active="yes"/>
 <layer number="41" name="tRestrict" color="4" fill="10" visible="no" active="yes"/>
 <layer number="42" name="bRestrict" color="1" fill="10" visible="no" active="yes"/>
 <layer number="43" name="vRestrict" color="2" fill="10" visible="no" active="yes"/>
 <layer number="44" name="Drills" color="7" fill="1" visible="no" active="yes"/>
-<layer number="45" name="Holes" color="7" fill="1" visible="yes" active="yes"/>
+<layer number="45" name="Holes" color="7" fill="1" visible="no" active="yes"/>
 <layer number="46" name="Milling" color="3" fill="1" visible="no" active="yes"/>
 <layer number="47" name="Measures" color="7" fill="1" visible="no" active="yes"/>
-<layer number="48" name="Document" color="7" fill="1" visible="yes" active="yes"/>
+<layer number="48" name="Document" color="7" fill="1" visible="no" active="yes"/>
 <layer number="49" name="Reference" color="7" fill="1" visible="no" active="yes"/>
 <layer number="50" name="dxf" color="7" fill="1" visible="no" active="yes"/>
@@
 <text x="30.2" y="1.7" size="1.01" layer="109" font="vector" ratio="15" rot="MR0"></text>
 <hole x="3.1" y="3.3" drill="3.2"/>
-<rectangle x1="19.7" y1="6.5" x2="21.2" y2="8" layer="30"/>
 <text x="34.67" y="2.57" size="0.8128" layer="108" font="vector" ratio="15">ext 5V</text>
 <text x="2" y="6.4" size="1.016" layer="1" font="vector" ratio="15" rot="R90">1</text>
 <text x="2" y="8.2" size="1.016" layer="16" font="vector" ratio="15" rot="R90">2</text>
-<text x="71.7" y="7.53" size="0.8128" layer="109" font="vector" ratio="15" rot="MR90">github.com/rodan/lemidi</text>
-<text x="73.13" y="7.55" size="0.8128" layer="109" font="vector" ratio="15" rot="MR90">Petre Rodan 201901 rev1</text>
+<text x="69.7" y="13.13" size="0.8128" layer="109" font="vector" ratio="15" rot="MR90">github.com/rodan/lemidi</text>
+<text x="71.13" y="13.15" size="0.8128" layer="109" font="vector" ratio="15" rot="MR90">Petre Rodan 201901 rev1</text>
 <text x="2.23" y="36.83" size="0.8128" layer="109" font="vector" ratio="15" rot="MR270">debug</text>
 <wire x1="1.55" y1="6.35" x2="1.55" y2="9.15" width="1.6764" layer="41"/>
-<rectangle x1="17.8" y1="5.1" x2="21.8" y2="9.4" layer="30"/>
-<text x="46" y="0.6" size="0.8128" layer="108" ratio="15">J1</text>
+<text x="39.6" y="0.6" size="0.8128" layer="108" ratio="15">J1</text>
 <text x="38.43" y="36.83" size="0.8128" layer="109" font="vector" ratio="15" rot="MR270">tp5</text>
 <text x="38.43" y="33.03" size="0.8128" layer="109" font="vector" ratio="15" rot="MR270">tp4</text>
@@
 <text x="9.83" y="23.83" size="0.8128" layer="109" font="vector" ratio="15" rot="MR270">tp7</text>
 <text x="5.23" y="9.63" size="0.8128" layer="109" font="vector" ratio="15" rot="MR270">tp1</text>
-<text x="48.9" y="25.07" size="0.8128" layer="109" font="vector" ratio="15" rot="MR270">tp1 - gnd
+<text x="41.3" y="21.87" size="0.8128" layer="109" font="vector" ratio="15" rot="MR270">tp1 - gnd
 tp2 - gnd
 tp3 - mosi
@@
 <wire x1="49.6" y1="1.9" x2="50" y2="1.9" width="0.254" layer="109"/>
 <wire x1="50" y1="1.9" x2="50.8" y2="2.7" width="0.254" layer="109"/>
-<wire x1="50.8" y1="16.5" x2="50.8" y2="25.5" width="0.254" layer="109"/>
-<wire x1="40" y1="15.7" x2="49.6" y2="15.7" width="0.254" layer="109"/>
-<wire x1="40" y1="25.5" x2="49.6" y2="25.5" width="0.254" layer="109"/>
-<wire x1="49.6" y1="25.5" x2="50.8" y2="25.5" width="0.254" layer="109"/>
-<text x="50" y="20.4" size="0.4064" layer="109" font="vector" ratio="15" rot="R270">test points</text>
-<wire x1="49.6" y1="15.7" x2="49.6" y2="25.5" width="0.1" layer="109"/>
-<wire x1="40" y1="25.5" x2="40" y2="15.7" width="0.254" layer="109"/>
-<wire x1="49.6" y1="15.7" x2="50" y2="15.7" width="0.254" layer="109"/>
-<wire x1="50" y1="15.7" x2="50.8" y2="16.5" width="0.254" layer="109"/>
+<wire x1="43.2" y1="13.3" x2="43.2" y2="22.3" width="0.254" layer="109"/>
+<wire x1="32.4" y1="12.5" x2="42" y2="12.5" width="0.254" layer="109"/>
+<wire x1="32.4" y1="22.3" x2="42" y2="22.3" width="0.254" layer="109"/>
+<wire x1="42" y1="22.3" x2="43.2" y2="22.3" width="0.254" layer="109"/>
+<text x="42.4" y="17.2" size="0.4064" layer="109" font="vector" ratio="15" rot="R270">test points</text>
+<wire x1="42" y1="12.5" x2="42" y2="22.3" width="0.1" layer="109"/>
+<wire x1="32.4" y1="22.3" x2="32.4" y2="12.5" width="0.254" layer="109"/>
+<wire x1="42" y1="12.5" x2="42.4" y2="12.5" width="0.254" layer="109"/>
+<wire x1="42.4" y1="12.5" x2="43.2" y2="13.3" width="0.254" layer="109"/>
 <text x="9.8" y="30.3" size="0.8128" layer="109" font="vector" ratio="15" rot="MR90">tx[]</text>
 <wire x1="17.6" y1="32.9" x2="17.6" y2="29.8" width="0.1" layer="109"/>
@@
 <element name="C4" library="rcl" package="C0805" value="1uF" x="29.35" y="8.6" rot="R90"/>
 <element name="C6" library="rcl" package="C0805" value="100nF" x="26.15" y="5.43"/>
-<element name="U$7" library="SparkFun" package="OSHW-LOGO-M" value="OSHW-LOGOM" x="73.01" y="3.35" rot="MR90"/>
+<element name="U$7" library="SparkFun" package="OSHW-LOGO-M" value="OSHW-LOGOM" x="71.01" y="8.95" rot="MR90"/>
 <element name="U$1" library="TI_MSP430_v16" package="PT48" value="MSP430F5510" x="28.8" y="28.8"/>
 <element name="C10" library="rcl" package="C0805" value="470nF" x="20.8" y="25" rot="R180"/>
@@
 <element name="C12" library="rcl" package="C0805" value="100nF" x="43.4" y="25.8"/>
 <element name="C13" library="rcl" package="C0805" value="100nF" x="43.4" y="34.4"/>
-<element name="J1" library="Simplex-Jumpers" package="SJ_3P" value="" x="44.9" y="2" rot="R180"/>
+<element name="J1" library="Simplex-Jumpers" package="SJ_3P" value="" x="41.9" y="2"/>
 <element name="C14" library="rcl" package="C0805" value="2.2nF" x="8.8" y="32.6" rot="R180"/>
 <element name="Y2" library="Simplex-FreqCtrl" package="CRYSTAL-SMD-11.4X4.35" value="12MHz 0.25% CL 16pF" x="28" y="18.4"/>
@@
 <via x="24.6" y="21.6" extent="1-16" drill="0.4"/>
 <via x="30.8" y="20.4" extent="1-16" drill="0.4"/>
-<via x="32.4" y="15.2" extent="1-16" drill="0.4"/>
+<via x="31.8" y="16.4" extent="1-16" drill="0.4"/>
 <via x="20.6" y="16" extent="1-16" drill="0.4"/>
 <contactref element="LED1" pad="C"/>
@@
 <wire x1="40.4" y1="3.6" x2="43" y2="3.6" width="0.6096" layer="1"/>
 <wire x1="43" y1="3.6" x2="43.4" y2="3.2" width="0.6096" layer="1"/>
-<wire x1="43.4" y1="3.2" x2="43.4" y2="2" width="0.6096" layer="1"/>
 <wire x1="49.2" y1="5.4" x2="47.4" y2="3.6" width="0.4064" layer="1"/>
 <wire x1="47.4" y1="3.6" x2="43.8" y2="3.6" width="0.4064" layer="1"/>
@@
 <wire x1="44.2" y1="25.95" x2="44.35" y2="25.8" width="0.4064" layer="1"/>
 <wire x1="42.8" y1="32.6" x2="42.8" y2="27.8" width="0.4064" layer="1"/>
+<wire x1="43.4" y1="2" x2="43.4" y2="3.2" width="0.6096" layer="1"/>
 </signal>
 <signal name="HIGH_MOSI">
@@
 </signal>
 <signal name="N$10">
-<contactref element="J1" pad="1"/>
 <contactref element="U$12" pad="P$1"/>
-<wire x1="44.9" y1="2" x2="48.9" y2="2.2" width="0.6096" layer="1"/>
 <wire x1="48.9" y1="2.2" x2="49.1" y2="2.6" width="0.6096" layer="1"/>
+<contactref element="J1" pad="3"/>
+<wire x1="44.9" y1="2" x2="49.1" y2="2" width="0.6096" layer="1"/>
+<wire x1="49.1" y1="2" x2="49.1" y2="2.6" width="0.6096" layer="1"/>
 </signal>
 <signal name="N$23">
 <contactref element="Q5" pad="2"/>
-<contactref element="J1" pad="3"/>
 <via x="40.4" y="2.2" extent="1-16" drill="0.4"/>
 <via x="31.6" y="11.2" extent="1-16" drill="0.4"/>
@@
 <wire x1="31.6" y1="11" x2="40.4" y2="2.2" width="0.6096" layer="16"/>
 <wire x1="31.6388" y1="11.1612" x2="31.6" y2="11.2" width="0.6096" layer="1"/>
-<wire x1="41.9" y1="2" x2="40.6" y2="2" width="0.6096" layer="1"/>
 <wire x1="40.6" y1="2" x2="40.4" y2="2.2" width="0.6096" layer="1"/>
 <wire x1="31.4388" y1="9.78413125" x2="31.4388" y2="11.0388" width="0.4064" layer="1"/>
 <wire x1="31.4388" y1="11.0388" x2="31.6" y2="11.2" width="0.4064" layer="1" curve="-90"/>
+<contactref element="J1" pad="1"/>
+<wire x1="40.6" y1="2" x2="41.9" y2="2" width="0.6096" layer="1"/>
 </signal>
 <signal name="N$24">
