File: hardware/lemidi.brd (EAGLE design)
At the start: 76 x 40 mm, 71 parts, among them Q1 IRLML6246, Q2 IRLML6246, Q3 IRLML6246, Q4 IRLML6246, Q5 si2305cd, U1 SPX5205 3v3, X3 debug, Y2 12MHz 0.25% CL 16pF, Y3 8MHz CL 18pF

Commit message: rev 2
Parts:
- Q1, Q2, Q3, Q4: value IRLML6246 -> PMBF170
Connections:
- removed net B4: OK1.10, U$10.14
- removed net B4_EN: Q2.1, U$2.5
- removed net J2X: U$10.11, U$4.5
- removed net J2Y: U$10.13, U$4.10
- new net B0: OK1.16, U$10.2
- new net B0_EN: Q4.1, U$2.8
- new net J0X: U$10.3, U$11.5
- new net J0Y: U$10.6, U$11.10
- net +3V3: now also U$6.8
- net B1: now also OK1.14, U$10.7; no longer OK1.16, U$10.2
- net B1_EN: now also Q3.1, U$2.7; no longer Q4.1, U$2.8
- net B2: now also OK1.12, U$10.10; no longer OK1.14, U$10.7
- net B2_EN: now also Q1.1, U$2.6; no longer Q3.1, U$2.7
- net B3: now also OK1.10, U$10.14; no longer OK1.12, U$10.10
- net B3_EN: now also Q2.1, U$2.5; no longer Q1.1, U$2.6
- net J1X: now also U$10.11, U$4.5; no longer U$10.3, U$11.5
- net J1Y: now also U$10.13, U$4.10; no longer U$10.6, U$11.10
Routing:
- net B4: track 36.6 -> 0.00 mm, vias 1 -> 0
- net B1: track 6.15 -> 36.7 mm
- net J0Y: track 0.00 -> 20.8 mm
- net J0X: track 0.00 -> 18.5 mm, vias 0 -> 3
- net J2Y: track 15.1 -> 0.00 mm
- net B2: track 36.7 -> 22.5 mm, vias 0 -> 1
- net B3: track 22.5 -> 36.6 mm
- net J2X: track 11.9 -> 0.00 mm
- net J1X: track 18.5 -> 11.9 mm, vias 3 -> 0
- net B0_EN: track 0.00 -> 6.17 mm
- net B0: track 0.00 -> 6.15 mm
- net J1Y: track 20.8 -> 15.1 mm
- net +3V3: track 105.4 -> 110.6 mm, vias 6 -> 8
- net B4_EN: track 3.86 -> 0.00 mm
- net B1_EN: track 6.17 -> 4.31 mm
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Other:
- board text added: "Petre Rodan 201901 rev 2"
- board text removed: "Petre Rodan 201901 rev1"
Changed lines of the file:
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@@
 <text x="2" y="8.2" size="1.016" layer="16" font="vector" ratio="15" rot="R90">2</text>
 <text x="69.7" y="13.13" size="0.8128" layer="109" font="vector" ratio="15" rot="MR90">github.com/rodan/lemidi</text>
-<text x="71.13" y="13.15" size="0.8128" layer="109" font="vector" ratio="15" rot="MR90">Petre Rodan 201901 rev1</text>
+<text x="71.13" y="13.15" size="0.8128" layer="109" font="vector" ratio="15" rot="MR90">Petre Rodan 201901 rev 2</text>
 <text x="2.23" y="36.83" size="0.8128" layer="109" font="vector" ratio="15" rot="MR270">debug</text>
 <wire x1="1.55" y1="6.35" x2="1.55" y2="9.15" width="1.6764" layer="41"/>
@@
 <attribute name="OC_FARNELL" value="unknown" x="50.6" y="10" size="1.778" layer="27" display="off"/>
 </element>
-<element name="Q2" library="Simplex-DiscreteSemi" package="SOT23-3" value="IRLML6246" x="34.4" y="13.2" rot="R180"/>
+<element name="Q2" library="Simplex-DiscreteSemi" package="SOT23-3" value="PMBF170" x="34.4" y="13.2" rot="R180"/>
 <element name="R26" library="rcl" package="R0805W" value="820" x="37.6" y="8.6" rot="R270"/>
-<element name="Q1" library="Simplex-DiscreteSemi" package="SOT23-3" value="IRLML6246" x="37.6" y="13.2" rot="R180"/>
+<element name="Q1" library="Simplex-DiscreteSemi" package="SOT23-3" value="PMBF170" x="37.6" y="13.2" rot="R180"/>
 <element name="R1" library="rcl" package="R0805W" value="820" x="39.8" y="8.6" rot="R270"/>
-<element name="Q3" library="Simplex-DiscreteSemi" package="SOT23-3" value="IRLML6246" x="40.8" y="13.2" rot="R180"/>
+<element name="Q3" library="Simplex-DiscreteSemi" package="SOT23-3" value="PMBF170" x="40.8" y="13.2" rot="R180"/>
 <element name="R3" library="rcl" package="R0805W" value="820" x="42" y="8.6" rot="R270"/>
-<element name="Q4" library="Simplex-DiscreteSemi" package="SOT23-3" value="IRLML6246" x="44" y="13.2" rot="R180"/>
+<element name="Q4" library="Simplex-DiscreteSemi" package="SOT23-3" value="PMBF170" x="44" y="13.2" rot="R180"/>
 <element name="R4" library="rcl" package="R0805W" value="820" x="44.2" y="8.6" rot="R270"/>
 <element name="C2" library="rcl" package="C0805" value="27pF" x="38.2" y="37.2" rot="R180"/>
@@
 <wire x1="36" y1="25" x2="36.4" y2="24.5" width="0.4064" layer="1"/>
 <wire x1="39" y1="24.5" x2="39.8" y2="25.2" width="0.4064" layer="1"/>
-<wire x1="39.8" y1="25.2" x2="39.8" y2="33" width="0.4064" layer="1"/>
+<wire x1="39.8" y1="25.2" x2="39.8" y2="27.2" width="0.4064" layer="1"/>
+<wire x1="39.8" y1="27.2" x2="39.8" y2="33" width="0.4064" layer="1"/>
 <wire x1="39.8" y1="33" x2="39.15" y2="33.65" width="0.4064" layer="1"/>
 <wire x1="39.15" y1="33.65" x2="39.15" y2="34.4" width="0.4064" layer="1"/>
@@
 <wire x1="15.26" y1="26.74" x2="15.06" y2="26.74" width="0.3048" layer="1"/>
 <wire x1="36.4" y1="24.5" x2="39" y2="24.5" width="0.4064" layer="1"/>
+<contactref element="U$6" pad="8"/>
+<wire x1="39.8" y1="27.2" x2="40.6" y2="27.2" width="0.3048" layer="1"/>
+<wire x1="40.6" y1="27.2" x2="40.8" y2="27.4" width="0.3048" layer="1"/>
+<via x="40.8" y="27.4" extent="1-16" drill="0.4"/>
+<via x="44.2" y="27.8" extent="1-16" drill="0.4"/>
+<wire x1="40.8" y1="27.4" x2="43.8" y2="27.4" width="0.3048" layer="16"/>
+<wire x1="43.8" y1="27.4" x2="44.2" y2="27.8" width="0.3048" layer="16"/>
+<wire x1="44.15" y1="28.3" x2="44.15" y2="27.85" width="0.3048" layer="1"/>
+<wire x1="44.15" y1="27.85" x2="44.2" y2="27.8" width="0.3048" layer="1"/>
 </signal>
 <signal name="N$6">
@@
 <wire x1="47.335" y1="13.2" x2="47.36" y2="13.175" width="0.3048" layer="1"/>
 </signal>
-<signal name="B1_EN">
+<signal name="B0_EN">
 <contactref element="Q4" pad="1"/>
 <contactref element="U$2" pad="8"/>
@@
 <wire x1="44.95" y1="15.25" x2="44.95" y2="14.2" width="0.3048" layer="1"/>
 </signal>
-<signal name="B2_EN">
+<signal name="B1_EN">
 <contactref element="Q3" pad="1"/>
 <contactref element="U$2" pad="7"/>
@@
 <wire x1="41.75" y1="15.25" x2="41.75" y2="14.2" width="0.3048" layer="1"/>
 </signal>
-<signal name="B3_EN">
+<signal name="B2_EN">
 <contactref element="Q1" pad="1"/>
 <contactref element="U$2" pad="6"/>
@@
 <wire x1="38.55" y1="15.75" x2="38.55" y2="14.2" width="0.3048" layer="1"/>
 </signal>
-<signal name="B4_EN">
+<signal name="B3_EN">
 <contactref element="Q2" pad="1"/>
 <contactref element="U$2" pad="5"/>
@@
 <wire x1="36.725" y1="15.6" x2="37.925" y2="16.8" width="0.3048" layer="1"/>
 </signal>
-<signal name="B1">
+<signal name="B0">
 <contactref element="OK1" pad="16"/>
 <contactref element="U$10" pad="2"/>
@@
 <wire x1="59.32" y1="13" x2="59.37" y2="13.05" width="0.4064" layer="1"/>
 </signal>
-<signal name="B2">
+<signal name="B1">
 <contactref element="OK1" pad="14"/>
 <contactref element="U$10" pad="7"/>
@@
 <wire x1="64.1" y1="26.9" x2="59.37" y2="26.9" width="0.4064" layer="1"/>
 </signal>
-<signal name="B3">
+<signal name="B2">
 <contactref element="OK1" pad="12"/>
 <contactref element="U$10" pad="10"/>
@@
 <wire x1="62.245" y1="14.4" x2="65.8" y2="14.4" width="0.4064" layer="16"/>
 </signal>
-<signal name="B4">
+<signal name="B3">
 <contactref element="OK1" pad="10"/>
 <contactref element="U$10" pad="14"/>
@@
 <wire x1="56.07" y1="29.67" x2="55.8" y2="29.4" width="0.4064" layer="16"/>
 </signal>
-<signal name="J1X">
+<signal name="J0X">
 <contactref element="U$10" pad="3"/>
 <contactref element="U$11" pad="5"/>
@@
 <wire x1="53.4" y1="29.2" x2="54.6" y2="28" width="0.4064" layer="1"/>
 </signal>
-<signal name="J1Y">
+<signal name="J0Y">
 <contactref element="U$10" pad="6"/>
 <contactref element="U$11" pad="10"/>
@@
 <wire x1="52.28" y1="37.08" x2="52.28" y2="35.73" width="0.4064" layer="1"/>
 </signal>
-<signal name="J2X">
+<signal name="J1X">
 <contactref element="U$10" pad="11"/>
 <contactref element="U$4" pad="5"/>
@@
 <wire x1="62.205" y1="17.2" x2="62.21" y2="17.205" width="0.4064" layer="1"/>
 </signal>
-<signal name="J2Y">
+<signal name="J1Y">
 <contactref element="U$10" pad="13"/>
 <contactref element="U$4" pad="10"/>
