File: hardware/lemidi.sch (EAGLE design)
At the start: 66 parts, among them Q1 IRLML6246, Q2 IRLML6246, Q3 IRLML6246, Q4 IRLML6246, U1 SPX5205 3v3, X1 MOLEX_2HORIZONTAL, X3 MOLEX_6HORIZONTAL, Y1 32768Hz CFPX-217 12.5pF, Y2 12MHz 0.25%, Y3 8MHz

Commit message: happy new year
Parts:
- removed C23, C24: 22pF, rcl:C-EUC0805
- removed Y1: 32768Hz CFPX-217 12.5pF, Simplex-FreqCtrl:CRYSTAL3.2X1.5
Connections:
- net N$1 renamed 12MHZ_XO
- net N$3 renamed 12MHX_XI
- removed net N$25: C24.1, U$1.9, Y1.1
- removed net N$26: C23.1, U$1.8, Y1.2
- removed net VIN: C3.1, C6.1, U1.EN, U1.IN
- new net N$1: LED1.A, R6.2
- new net N$20: U$1.20, U$2.2
- new net N$21: U$1.21, U$2.1
- new net N$3: U$1.18, U$2.4
- net +5V: now also C3.1, C6.1, U1.EN, U1.IN
- net B1_EN: now also U$2.8
- net B2_EN: now also U$2.7
- net B3_EN: now also U$2.6
- net B4_EN: now also U$2.5
- net GND: now also LED1.C, LED2.C, LED3.C; no longer C23.2, C24.2, R10.2, R6.2, R9.2
- net N$11: now also LED3.A, R10.2; no longer LED3.C, R10.1
- net N$4: now also LED2.A, R9.2; no longer LED2.C, R9.1
- net N$8: now also U$1.19, U$2.3; no longer LED1.C, R6.1
- net STATUS: now also R6.1; no longer LED1.A
- net USB_GPX: now also U$1.15
- net USB_INT: now also U$1.14
- net USB_ST1: now also R9.1; no longer LED2.A
- net USB_ST2: now also R10.1; no longer LED3.A
Other:
- moved on the sheet: C1, C10, C11, C12, C13, C14, C15, C16, C17, C18, C19, C2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

Commit message: latest
Parts:
- LED3: value green -> red
- U$10: value ADAM_TECH-DSUB_DA-15 -> DA-15
- X1: value MOLEX_2HORIZONTAL -> optional 5V input
- X3: value MOLEX_6HORIZONTAL -> debug
Connections:
- removed net CSJ1: U$6.A1
- removed net CSJ2: U$6.A2
- removed net USB_CS: U$3.!SS
- new net CS_J1: U$1.36, U$6.A1
- new net CS_J2: U$1.35, U$6.A2
- new net CS_USB: U$1.29, U$3.!SS
- net HIGH_MOSI: now also U$6.Y4; no longer U$6.Y3
- net HIGH_SCLK: now also U$6.Y3; no longer U$6.Y4
- net MOSI: now also U$6.A4; no longer U$6.A3
- net SCLK: now also U$6.A3; no longer U$6.A4
- net USB_RES: now also U$1.2
Other:
- note added: "digital output pins: - MOSI - MISO - SCLK - CS_USB - CS_J1 - CS_J2 - USB_RES - STATUS LED"
- note removed: "digital output pins: - MOSI - MISO - SCLK - USB_CS - CS_POT1 - CS_POT2 - USB_RES - STATUS LED"
- moved on the sheet: C1, C10, C15, C16, C17, C18, C19, C2, C3, C4, C5, C6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

Commit message: latest
Parts:
- added C21: 100nF, rcl:C-EUC0805
- added TP4, TP5: TPTP12R, testpad:TPTP12R
Connections:
- removed net STATUS: R6.1, TP6.TP
- new net USB_ST3: R6.1, U$3.GPOUT2
- net +3V3: now also C21.2
- net CS_USB: now also TP5.TP
- net GND: now also C21.1, TP6.TP
- net MISO: now also TP3.TP
- net MOSI: now also TP4.TP
- net SCLK: now also TP2.TP
- net USB_GPX: now also U$1.14; no longer U$1.15
- net USB_INT: now also U$1.15; no longer U$1.14
- net USB_ST1: no longer TP2.TP
- net USB_ST2: no longer TP3.TP
Other:
- moved on the sheet: LED1, LED2, LED3, R10, R6, R9, TP2, TP3, TP6

Commit message: ERC pass
Parts:
- C14: value 10nF -> 2.2nF
Connections:
- removed net N$10: U$3.GND
- net GND: now also U$3.GND
Changed lines of the file:
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@@
 <part name="U$11" library="Simplex-Jumpers" deviceset="SJ_3P" device=""/>
 <part name="SUPPLY9" library="supply2" deviceset="+5V" device=""/>
-<part name="C14" library="rcl" deviceset="C-EU" device="C0805" value="10nF"/>
+<part name="C14" library="rcl" deviceset="C-EU" device="C0805" value="2.2nF"/>
 <part name="GND31" library="SparkFun" deviceset="GND" device=""/>
 <part name="Y2" library="Simplex-FreqCtrl" deviceset="CRYSTAL" device="" value="12MHz 0.25%"/>
@@
 <wire x1="187.96" y1="15.24" x2="187.96" y2="17.78" width="0.1524" layer="91"/>
 </segment>
+<segment>
+<pinref part="U$3" gate="G$1" pin="GND"/>
+<pinref part="GND38" gate="1" pin="GND"/>
+<wire x1="101.6" y1="144.78" x2="116.84" y2="144.78" width="0.1524" layer="91"/>
+<wire x1="116.84" y1="144.78" x2="116.84" y2="139.7" width="0.1524" layer="91"/>
+</segment>
 </net>
 <net name="+3V3" class="0">
@@
 <wire x1="208.28" y1="139.7" x2="200.66" y2="139.7" width="0.1524" layer="91"/>
 <wire x1="200.66" y1="139.7" x2="200.66" y2="137.16" width="0.1524" layer="91"/>
+<junction x="208.28" y="139.7"/>
 </segment>
 <segment>
@@
 </segment>
 </net>
-<net name="N$10" class="0">
-<segment>
-<pinref part="GND38" gate="1" pin="GND"/>
-<pinref part="U$3" gate="G$1" pin="GND"/>
-<wire x1="101.6" y1="144.78" x2="116.84" y2="144.78" width="0.1524" layer="91"/>
-<wire x1="116.84" y1="144.78" x2="116.84" y2="139.7" width="0.1524" layer="91"/>
-</segment>
-</net>

Commit message: 1st cleanup
Parts:
- added TP7: TPTP12R, testpad:TPTP12R
Connections:
- net CS_J1: now also TP7.TP
Changed lines of the file:
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@@
 <part name="TP6" library="testpad" deviceset="TP" device="TP12R" value=""/>
 <part name="GND46" library="SparkFun" deviceset="GND" device=""/>
+<part name="TP7" library="testpad" deviceset="TP" device="TP12R" value=""/>
 </parts>
 <sheets>
@@
 <instance part="TP6" gate="G$1" x="187.96" y="20.32"/>
 <instance part="GND46" gate="1" x="187.96" y="12.7"/>
+<instance part="TP7" gate="G$1" x="167.64" y="45.72" rot="R270"/>
 </instances>
 <busses>
@@
 <segment>
 <pinref part="U$1" gate="G$1" pin="36"/>
-<wire x1="154.94" y1="45.72" x2="157.48" y2="45.72" width="0.1524" layer="91"/>
+<wire x1="154.94" y1="45.72" x2="165.1" y2="45.72" width="0.1524" layer="91"/>
 <label x="157.48" y="45.72" size="1.778" layer="95"/>
-</segment>
-<segment>
+<pinref part="TP7" gate="G$1" pin="TP"/>
+</segment>
+<segment>

Commit message: 2nd cleanup
Connections:
- removed net CS_J1: TP7.TP, U$1.36, U$6.A1
- new net TP5: TP5.TP, U$1.36, U$6.A1
- net CS_USB: now also TP6.TP; no longer TP5.TP
- net GND: now also TP2.TP; no longer TP6.TP
- net MISO: now also TP7.TP; no longer TP3.TP
- net MOSI: now also TP3.TP; no longer TP4.TP
- net SCLK: now also TP4.TP; no longer TP2.TP
Other:
- moved on the sheet: TP2, TP3, TP4, TP5, TP6, TP7
Changed lines of the file:
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@@
 <part name="C21" library="rcl" deviceset="C-EU" device="C0805" value="100nF"/>
 <part name="GND33" library="SparkFun" deviceset="GND" device=""/>
+<part name="TP4" library="testpad" deviceset="TP" device="TP12R" value=""/>
+<part name="TP7" library="testpad" deviceset="TP" device="TP12R" value=""/>
+<part name="TP3" library="testpad" deviceset="TP" device="TP12R" value=""/>
+<part name="TP6" library="testpad" deviceset="TP" device="TP12R" value=""/>
 <part name="TP2" library="testpad" deviceset="TP" device="TP12R" value=""/>
-<part name="TP3" library="testpad" deviceset="TP" device="TP12R" value=""/>
-<part name="TP4" library="testpad" deviceset="TP" device="TP12R" value=""/>
+<part name="GND46" library="SparkFun" deviceset="GND" device=""/>
 <part name="TP5" library="testpad" deviceset="TP" device="TP12R" value=""/>
-<part name="TP6" library="testpad" deviceset="TP" device="TP12R" value=""/>
-<part name="GND46" library="SparkFun" deviceset="GND" device=""/>
-<part name="TP7" library="testpad" deviceset="TP" device="TP12R" value=""/>
 </parts>
 <sheets>
@@
 <instance part="C21" gate="G$1" x="187.96" y="198.12" rot="R180"/>
 <instance part="GND33" gate="1" x="187.96" y="193.04"/>
-<instance part="TP2" gate="G$1" x="167.64" y="35.56" rot="R270"/>
-<instance part="TP3" gate="G$1" x="167.64" y="33.02" rot="R270"/>
-<instance part="TP4" gate="G$1" x="167.64" y="30.48" rot="R270"/>
-<instance part="TP5" gate="G$1" x="167.64" y="27.94" rot="R270"/>
-<instance part="TP6" gate="G$1" x="187.96" y="20.32"/>
+<instance part="TP4" gate="G$1" x="167.64" y="35.56" rot="R270"/>
+<instance part="TP7" gate="G$1" x="167.64" y="33.02" rot="R270"/>
+<instance part="TP3" gate="G$1" x="167.64" y="30.48" rot="R270"/>
+<instance part="TP6" gate="G$1" x="167.64" y="27.94" rot="R270"/>
+<instance part="TP2" gate="G$1" x="187.96" y="20.32"/>
 <instance part="GND46" gate="1" x="187.96" y="12.7"/>
-<instance part="TP7" gate="G$1" x="167.64" y="45.72" rot="R270"/>
+<instance part="TP5" gate="G$1" x="167.64" y="45.72" rot="R270"/>
 </instances>
 <busses>
@@
 <segment>
 <pinref part="GND46" gate="1" pin="GND"/>
-<pinref part="TP6" gate="G$1" pin="TP"/>
+<pinref part="TP2" gate="G$1" pin="TP"/>
 <wire x1="187.96" y1="15.24" x2="187.96" y2="17.78" width="0.1524" layer="91"/>
 </segment>
@@
 <pinref part="U$1" gate="G$1" pin="30"/>
 <label x="157.48" y="30.48" size="1.778" layer="95"/>
-<pinref part="TP4" gate="G$1" pin="TP"/>
+<pinref part="TP3" gate="G$1" pin="TP"/>
 <wire x1="154.94" y1="30.48" x2="165.1" y2="30.48" width="0.1524" layer="91"/>
 </segment>
@@
 <pinref part="U$1" gate="G$1" pin="31"/>
 <label x="157.48" y="33.02" size="1.778" layer="95"/>
-<pinref part="TP3" gate="G$1" pin="TP"/>
+<pinref part="TP7" gate="G$1" pin="TP"/>
 <wire x1="154.94" y1="33.02" x2="165.1" y2="33.02" width="0.1524" layer="91"/>
 </segment>
@@
 <pinref part="U$1" gate="G$1" pin="32"/>
 <label x="157.48" y="35.56" size="1.778" layer="95"/>
-<pinref part="TP2" gate="G$1" pin="TP"/>
+<pinref part="TP4" gate="G$1" pin="TP"/>
 <wire x1="154.94" y1="35.56" x2="165.1" y2="35.56" width="0.1524" layer="91"/>
 </segment>
@@
 </segment>
 </net>
-<net name="CS_J1" class="0">
+<net name="TP5" class="0">
 <segment>
 <pinref part="U$1" gate="G$1" pin="36"/>
 <wire x1="154.94" y1="45.72" x2="165.1" y2="45.72" width="0.1524" layer="91"/>
 <label x="157.48" y="45.72" size="1.778" layer="95"/>
-<pinref part="TP7" gate="G$1" pin="TP"/>
+<pinref part="TP5" gate="G$1" pin="TP"/>
 </segment>
 <segment>
@@
 <pinref part="U$1" gate="G$1" pin="29"/>
 <label x="157.48" y="27.94" size="1.778" layer="95"/>
-<pinref part="TP5" gate="G$1" pin="TP"/>
+<pinref part="TP6" gate="G$1" pin="TP"/>
 <wire x1="154.94" y1="27.94" x2="165.1" y2="27.94" width="0.1524" layer="91"/>
 </segment>

Commit message: 3rd cleanup
Parts:
- removed X1: optional 5V input, Simplex-Connectors:MOLEX_2HORIZONTAL
- added JP1: external 5v, SparkFun-Connectors:M02PTH
Connections:
- net 5V_EXT: now also JP1.1; no longer X1.1
- net GND: now also JP1.2; no longer X1.2
Changed lines of the file:
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@@
 <layer number="97" name="Info" color="7" fill="1" visible="yes" active="yes"/>
 <layer number="98" name="Guide" color="6" fill="1" visible="yes" active="yes"/>
+<layer number="99" name="SpiceOrder" color="7" fill="1" visible="yes" active="yes"/>
 <layer number="100" name="Muster" color="7" fill="1" visible="no" active="no"/>
 <layer number="101" name="Patch_Top" color="12" fill="4" visible="yes" active="yes"/>
@@
 <part name="C3" library="rcl" deviceset="C-EU" device="C0805" value="10uF"/>
 <part name="X3" library="Simplex-Connectors" deviceset="MOLEX_6" device="HORIZONTAL" value="debug"/>
-<part name="X1" library="Simplex-Connectors" deviceset="MOLEX_2" device="HORIZONTAL" value="optional 5V input"/>
 <part name="R7" library="rcl" deviceset="R-EU_" device="R0805W" value="4k7"/>
 <part name="R8" library="rcl" deviceset="R-EU_" device="R0805W" value="4k7"/>
@@
 <part name="GND46" library="SparkFun" deviceset="GND" device=""/>
 <part name="TP5" library="testpad" deviceset="TP" device="TP12R" value=""/>
+<part name="JP1" library="SparkFun-Connectors" deviceset="M02" device="PTH" value="external 5v"/>
 </parts>
 <sheets>
@@
 <instance part="C3" gate="G$1" x="66.04" y="193.04"/>
 <instance part="X3" gate="G$1" x="274.32" y="22.86"/>
-<instance part="X1" gate="G$1" x="312.42" y="20.32"/>
 <instance part="R7" gate="G$1" x="259.08" y="33.02" rot="MR270"/>
 <instance part="R8" gate="G$1" x="254" y="33.02" rot="MR270"/>
@@
 <instance part="GND46" gate="1" x="187.96" y="12.7"/>
 <instance part="TP5" gate="G$1" x="167.64" y="45.72" rot="R270"/>
+<instance part="JP1" gate="G$1" x="317.5" y="20.32" rot="R180"/>
 </instances>
 <busses>
@@
 <wire x1="304.8" y1="17.78" x2="304.8" y2="10.16" width="0.1524" layer="91"/>
 <wire x1="304.8" y1="17.78" x2="309.88" y2="17.78" width="0.1524" layer="91"/>
-<pinref part="X1" gate="G$1" pin="2"/>
+<pinref part="JP1" gate="G$1" pin="2"/>
 </segment>
 <segment>
@@
 <net name="5V_EXT" class="0">
 <segment>
-<pinref part="X1" gate="G$1" pin="1"/>
 <wire x1="309.88" y1="20.32" x2="304.8" y2="20.32" width="0.1524" layer="91"/>
 <label x="297.18" y="20.32" size="1.778" layer="95"/>
-</segment>
-<segment>
+<pinref part="JP1" gate="G$1" pin="1"/>
+</segment>
+<segment>
